File: PCB/robo-con-Ethernet-v2/robo-con-Ethernet-v2.kicad_sch (KiCad schematic)
At the start: 98 parts, among them J1 Conn_01x04, J2 Conn_01x04, J4 RJ45_Bel_SI-60062-F, J5 Conn_01x02, J7 Conn_01x06, J8 Conn_01x06, SW1 SW_Push, SW2 SW_Push, U1 STM32G474RCTx, U10 MCP73831-2-OT, U11 LM66100DCK, U15 LM66100DCK, U18 USB_Type-C, U3 W5500, U5 RKJXV122400R, U6 NJM2884U1-33, U7 RKJXV122400R, U8 TMHU28, U9 TMHU28, Y2 XRCGB25M000FFS1AR0

Commit message: update pcb
Parts:
- removed J1: Conn_01x04, Connector_PinSocket_2.54mm:PinSocket_1x04_P2.54mm_Horizontal, symbol Connector_Generic:Conn_01x04
- removed J7, J8: Conn_01x06, Connector_JST:JST_ZH_B6B-ZR_1x06_P1.50mm_Vertical, symbol Connector_Generic:Conn_01x06
- removed R5: MNR04M0ABJ103, My_Library:MNR04M0ABJ103, symbol My_Library:MNR04M0ABJ103
- removed U8, U9: TMHU28, My_Library:TMHU28, symbol My_Library:TMHU28
- added D16: G, LED_SMD:LED_0603_1608Metric_Pad1.05x0.95mm_HandSolder, symbol Device:LED_Small
- added D17: R, LED_SMD:LED_0603_1608Metric_Pad1.05x0.95mm_HandSolder, symbol Device:LED_Small
- added J1, J3: Conn_01x05, Connector_JST:JST_ZH_B5B-ZR_1x05_P1.50mm_Vertical, symbol Connector_Generic:Conn_01x05
- added R12, R13, R14, R35, R36: 1k, Resistor_SMD:R_0402_1005Metric_Pad0.72x0.64mm_HandSolder, symbol Device:R_Small
- added SW3, SW4: SW_Push, My_Library:SKHHLPA010, symbol Switch:SW_Push
- added SW5: SW_Push_SPDT, My_Library:4MS1R202M6QES, symbol Switch:SW_Push_SPDT
- added SW6, SW7: SW_Push_SPDT, My_Library:8MS8P1B05VS2QES-C13, symbol Switch:SW_Push_SPDT
- R24: value 2.2k -> 4k; footprint Resistor_SMD:R_0402_1005Metric_Pad0.72x0.64mm_HandSolder -> Resistor_SMD:R_0603_1608Metric_Pad0.98x0.95mm_HandSolder
Connections:
- net +3.3V: now also J1.1 (Pin_1), J3.5 (Pin_5), R12.1, R13.1, R14.1, R35.1, SW3.2, SW4.2, SW6.1 (A), SW7.1 (A)
- net +5V: now also SW5.1 (A); no longer R79.1
- net GND: now also R36.2, SW5.3 (C), SW6.3 (C), SW7.3 (C); no longer U18.S1 (SHIELD)
- net LiPo_Observe: no longer U1.17 (PA3)
- net W5500_MISO: no longer U1.20 (PA6)
- net W5500_MOSI: no longer U1.21 (PA7)
- net W5500_SCLK: no longer U1.19 (PA5)
- net W5500_nCS: no longer U1.18 (PA4)
- net W5500_nINT: no longer U1.24 (PB0)
- net W5500_nRST: no longer U1.25 (PB1)
- net at R79.2: now also SW5.2 (B); no longer U6.1 (CONT)
- net at U3.43 (PMODE2): now also R14.2
- net at U3.44 (PMODE1): now also R13.2
- net at U3.45 (PMODE0): now also R12.2
- net Left_Button_1: no longer names the net of U1.51 (PA15)
- net Left_Button_2: no longer names the net of U1.52 (PC10)
- net Left_Button_3: no longer names the net of U1.53 (PC11)
- net Left_Button_4: no longer names the net of U1.54 (PC12)
- net Left_Lever_Switch_0: no longer names the net of U1.58 (PB5)
- net Left_Lever_Switch_1: no longer names the net of U1.60 (PB7)
- net Left_Lever_Switch_2: no longer names the net of U1.59 (PB6)
- net Left_Lever_Switch_3: no longer names the net of U1.56 (PB3)
- net Left_Lever_Switch_4: no longer names the net of U1.57 (PB4)
- net Left_Push_Stick renamed LP_STICK
- net LP_STICK: no longer U1.10 (PC2)
- net Left_X_Stick: no longer names the net of U1.8 (PC0)
- net Left_X_Stick: no longer U5.2 (X_shaft)
- net Left_Y_Stick: no longer names the net of U1.9 (PC1)
- net Left_Y_Stick: no longer U5.5 (Y_shaft)
- net Right_Button_5: no longer names the net of U1.35 (PB13)
- net Right_Button_6: no longer names the net of U1.36 (PB14)
- net Right_Button_7: no longer names the net of U1.37 (PB15)
- net Right_Button_8: no longer names the net of U1.22 (PC4)
- net Right_Lever_Switch_0: no longer names the net of U1.40 (PC8)
- net Right_Lever_Switch_1: no longer names the net of U1.39 (PC7)
- net Right_Lever_Switch_2: no longer names the net of U1.38 (PC6)
- net Right_Lever_Switch_3: no longer names the net of U1.42 (PA8)
- net Right_Lever_Switch_4: no longer names the net of U1.41 (PC9)
- net Right_Push_Stick renamed RP_STICK
- net RP_STICK: no longer U1.11 (PC3)
- net Right_X_Stick: no longer names the net of U1.33 (PB11)
- net Right_X_Stick: no longer U7.2 (X_shaft)
- net Right_Y_Stick: no longer names the net of U1.34 (PB12)
- net Right_Y_Stick: no longer U7.5 (Y_shaft)
- net ST_LED_0: no longer names the net of U1.6 (PF1)
- net ST_LED_0: no longer R2.1
- net ST_LED_1: no longer names the net of U1.5 (PF0)
- net ST_LED_1: no longer R4.1
- net ST_LED_2: no longer names the net of U1.4 (PC15)
- net ST_LED_2: no longer R6.1
- net ST_LED_3: no longer names the net of U1.3 (PC14)
- net ST_LED_3: no longer R11.1
- net ST_LED_4: no longer names the net of U1.2 (PC13)
- net ST_LED_4: no longer R32.1
- net ST_LED_USB: no longer names the net of U1.44 (PA10)
- net ST_LED_USB: no longer R33.1
- net ST_LED_W5500: no longer names the net of U1.43 (PA9)
- net ST_LED_W5500: no longer R34.1
- net VBUS: no longer names the net of C12.1, FB1.2, U11.1 (VIN)
- net Wio-E5_RST: no longer names the net of U1.30 (PB10)
- new net: D17.1 (K), R36.1
- new net: D16.2 (A), R35.2
- new net L5_BUTTON: J3.4 (Pin_4)
- new net L6_BUTTON: J3.3 (Pin_3)
- new net L7_BUTTON: J3.2 (Pin_2)
- new net L8_BUTTON: J3.1 (Pin_1)
- new net LED0: R2.1
- new net LED1: R4.1
- new net LED2: R6.1
- new net LED3: R11.1
- new net LED4: R32.1
- new net LEDLiPo: D16.1 (K), D17.2 (A)
- new net LEDUSB: R33.1
- new net LEDW5500: R34.1
- new net LX_STICK: U5.2 (X_shaft)
- new net LY_STICK: U5.5 (Y_shaft)
- new net L_PUSH: SW3.1
- new net L_PUSH_UP: SW6.2 (B)
- new net R1_BUTTON: J1.2 (Pin_2)
- new net R2_BUTTON: J1.3 (Pin_3)
- new net R3_BUTTON: J1.4 (Pin_4)
- new net R4_BUTTON: J1.5 (Pin_5)
- new net RX_STICK: U7.2 (X_shaft)
- new net RY_STICK: U7.5 (Y_shaft)
- new net R_PUSH: SW4.1
- new net R_PUSH_UP: SW7.2 (B)
- new net V_ON: R79.1, U6.1 (CONT)
- no-connect marks 19 -> 18
Other:
- moved on the sheet: R79

Commit message: PCBのGNDビア打ち以外終了 iocファイルとの照合はまだ 明日やる
Connections:
- net +3.3V: now also J1.5 (Pin_5), J3.1 (Pin_1); no longer J1.1 (Pin_1), J3.5 (Pin_5)
- net L5_BUTTON: now also J3.2 (Pin_2), U1.41 (PC9); no longer J3.4 (Pin_4)
- net L6_BUTTON: now also U1.42 (PA8)
- net L7_BUTTON: now also J3.4 (Pin_4), U1.43 (PA9); no longer J3.2 (Pin_2)
- net L8_BUTTON: now also J3.5 (Pin_5), U1.44 (PA10); no longer J3.1 (Pin_1)
- net LED0: now also U1.52 (PC10)
- net LED1: now also U1.53 (PC11)
- net LED2: now also U1.54 (PC12)
- net LED3: now also U1.55 (PD2)
- net LED4: now also U1.56 (PB3)
- net LEDLiPo: now also U1.12 (PA0)
- net LEDUSB: now also U1.57 (PB4)
- net LEDW5500: now also U1.58 (PB5)
- net LP_STICK: now also U1.10 (PC2)
- net LX_STICK: now also U1.9 (PC1)
- net LY_STICK: now also U1.8 (PC0)
- net L_PUSH: now also U1.51 (PA15)
- net L_PUSH_UP: now also U1.40 (PC8)
- net LiPo_Observe: now also U1.17 (PA3)
- net R1_BUTTON: now also J1.4 (Pin_4), U1.23 (PC5); no longer J1.2 (Pin_2)
- net R2_BUTTON: now also U1.22 (PC4)
- net R3_BUTTON: now also J1.2 (Pin_2), U1.21 (PA7); no longer J1.4 (Pin_4)
- net R4_BUTTON: now also J1.1 (Pin_1), U1.20 (PA6); no longer J1.5 (Pin_5)
- net RP_STICK: now also U1.11 (PC3)
- net RX_STICK: now also U1.19 (PA5)
- net RY_STICK: now also U1.18 (PA4)
- net R_PUSH: now also U1.14 (PA2)
- net R_PUSH_UP: now also U1.13 (PA1)
- net W5500_MISO: now also U1.36 (PB14)
- net W5500_MOSI: now also U1.37 (PB15)
- net W5500_SCLK: now also U1.35 (PB13)
- net W5500_nCS: now also U1.34 (PB12)
- net W5500_nINT: now also U1.38 (PC6)
- net W5500_nRST: now also U1.39 (PC7)
- no-connect marks 18 -> 11

Commit message: ioc 比較済み
Connections:
- net L_PUSH_UP renamed L_PUSH_HOME
- net R_PUSH_UP renamed R_PUSH_HOME
- no-connect marks 11 -> 24
Changed lines of the file:
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@@
 	)
 	(no_connect
+		(at 62.23 74.93)
+	)
+	(no_connect
+		(at 97.79 107.95)
+	)
+	(no_connect
 		(at 297.18 80.01)
 	)
 	(no_connect
+		(at 97.79 133.35)
+	)
+	(no_connect
 		(at 320.04 69.85)
 	)
 	(no_connect
+		(at 62.23 120.65)
+	)
+	(no_connect
 		(at 242.57 172.72)
 	)
@@
 	)
 	(no_connect
+		(at 97.79 128.27)
+	)
+	(no_connect
+		(at 97.79 105.41)
+	)
+	(no_connect
+		(at 97.79 120.65)
+	)
+	(no_connect
+		(at 97.79 123.19)
+	)
+	(no_connect
+		(at 62.23 123.19)
+	)
+	(no_connect
+		(at 97.79 130.81)
+	)
+	(no_connect
 		(at 320.04 72.39)
 	)
 	(no_connect
+		(at 97.79 110.49)
+	)
+	(no_connect
+		(at 62.23 72.39)
+	)
+	(no_connect
 		(at 273.05 157.48)
 	)
@@
 	)
 	(no_connect
+		(at 62.23 118.11)
+	)
+	(no_connect
 		(at 273.05 162.56)
 	)
@@
 		)
 	)
-	(global_label "L_PUSH_UP"
+	(global_label "L_PUSH_HOME"
 		(shape input)
 		(at 62.23 105.41 180)
@@
 		)
 		(property "Intersheetrefs" "${INTERSHEET_REFS}"
-			(at 48.5405 105.41 0)
+			(at 45.8796 105.41 0)
 			(hide yes)
 			(show_name no)
@@
 		)
 	)
-	(global_label "R_PUSH_UP"
+	(global_label "R_PUSH_HOME"
 		(shape input)
 		(at 95.25 218.44 180)
@@
 		)
 		(property "Intersheetrefs" "${INTERSHEET_REFS}"
-			(at 81.3186 218.44 0)
+			(at 78.6577 218.44 0)
 			(hide yes)
 			(show_name no)
@@
 		)
 	)
-	(global_label "L_PUSH_UP"
+	(global_label "L_PUSH_HOME"
 		(shape input)
 		(at 58.42 218.44 180)
@@
 		)
 		(property "Intersheetrefs" "${INTERSHEET_REFS}"
-			(at 44.7305 218.44 0)
+			(at 42.0696 218.44 0)
 			(hide yes)
 			(show_name no)
@@
 		)
 	)
-	(global_label "R_PUSH_UP"
+	(global_label "R_PUSH_HOME"
 		(shape input)
 		(at 97.79 64.77 0)
@@
 		)
 		(property "Intersheetrefs" "${INTERSHEET_REFS}"
-			(at 111.7214 64.77 0)
+			(at 114.3823 64.77 0)
 			(hide yes)
 			(show_name no)
